Commit message: feat: 미아 탐지 및 고객센터 에스코트 파이프라인 추가
- myrobot_vision 패키지: YOLOv8 어린이 감지, 보호자 부재 판단, TTS 에스코트, 순찰 노드
- model_mover: Gazebo 내 인물 모델 배치 자동화
- Nav2 설정, vision launch, 인물 모델 리소스 추가

Co-Authored-By: Claude Sonnet 4.6 <noreply@anthropic.com>

File: src/myrobot/urdf/my_robot.urdf (robot description, URDF)
Before this commit: robot my_robot, 7 links, 6 joints
Links:
- added link depth_camera_link, mass 0.001; collision box size=0.01 0.01 0.01; visual box size=0.04 0.04 0.04
- link camera_link: mass None -> 0.001; geometry collision box size=0.01 0.01 0.01; visual box size=0.05 0.05 0.05
Joints:
- added joint depth_camera_joint: type fixed, parent base_link, child depth_camera_link, origin xyz=0.1 0.0 0.2 rpy=0 0 0
